Commit message: big push

File: URDF/Student_Arm.SLDASM/urdf/Student_Arm.SLDASM.urdf (robot description, URDF)
Before this commit: robot Student_Arm.SLDASM, 9 links, 8 joints
Links:
- link Gripper_Left: mass 0.0189723242002883 -> 0.0232588565708634
- link Gripper_Right: mass 0.0189723242002881 -> 0.0232588565708632
- link J1: mass 0.50399 -> 0.503990921516619
- link J2: mass 0.39279 -> 0.392763832529056
- link J3: mass 0.20982 -> 0.208448276188946
- link J4: mass 0.060711 -> 0.0607110395840995
- link J5: mass 0.053474 -> 0.0534742460950643
- link J6: mass 0.10498725932869 -> 0.101334847700238
Joints:
- joint GL: axis -1 0 0 -> 1 0 0; limit lower=0 upper=0 effort=0 velocity=0 -> lower=0 upper=0.057 effort=0 velocity=0
- joint GR: limit lower=0 upper=0 effort=0 velocity=0 -> lower=0 upper=0.057 effort=0 velocity=0; mimic (none) -> joint=GL multiplier=1 offset=0
- joint J1: axis 0 0 0 -> 0 1 0
- joint J2: axis 0 0 0 -> 0 0 -1; limit lower=0 upper=0 effort=0 velocity=0 -> lower=-1.4 upper=2.5 effort=0 velocity=0
- joint J3: limit (none) -> lower=-1.4 upper=1.8 effort=0 velocity=0; type continuous -> revolute
- joint J4: limit (none) -> lower=0 upper=0 effort=0 velocity=0; type continuous -> revolute
- joint J5: limit (none) -> lower=-0.75 upper=2.9 effort=0 velocity=0; type continuous -> revolute
- joint J6: limit (none) -> lower=0 upper=0 effort=0 velocity=0; type continuous -> revolute
